Commit message: Updated urdf file

File: neuronbot2_description/urdf/neuronbot2.urdf (robot description, URDF)
Before this commit: robot neuronbot2_description, 3 links, 2 joints
Links:
- added link base_footprint
- added link wheel_left_link, mass 2.8498940e-02; collision cylinder length=0.025 radius=0.075; visual cylinder length=0.025 radius=0.075
- added link wheel_right_link, mass 2.8498940e-02; collision cylinder length=0.025 radius=0.075; visual cylinder length=0.025 radius=0.075
- link base_link: mass 4.7982 -> 5; geometry collision box size=0.33 0.33 0.2; visual mesh filename=package://neuronbot2_description/meshes/neuronbot2/base_lin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
- link laser_frame: mass 0.17934 -> 0.2
Joints:
- added joint base_link_joint: type fixed, parent base_footprint, child base_link, origin xyz=0 0 0 rpy=0 0 0
- added joint l_wheel_joint: type continuous, parent base_link, child wheel_left_link, origin xyz=0.0 0.14 0.0745 rpy=1.57 0 0, axis 0 0 1
- added joint r_wheel_joint: type continuous, parent base_link, child wheel_right_link, origin xyz=0.0 -0.14 0.0745 rpy=1.57 0 0, axis 0 0 1
- joint imu_joint: origin xyz=0 0 0.11 rpy=0 0 1.57 -> xyz=0 0 0.11 rpy=0 0 0
- joint laser_frame_joint: origin xyz=0.001 0 0.31 rpy=0 0 3.14 -> xyz=0.125 0 0.33 rpy=0 0 3.14

Commit message: Added an unnecessary missing line

File: neuronbot2_description/urdf/neuronbot2.urdf (robot description, URDF)
Before this commit: robot neuronbot2_description, 6 links, 5 joints
Joints:
- joint imu_joint: axis (none) -> 0 0 0

Commit message: Update 3Ds model and urdf file for REAL Neuronbot2

File: neuronbot2_description/urdf/neuronbot2.urdf (robot description, URDF)
Before this commit: robot neuronbot2_description, 6 links, 5 joints
Links:
- link base_link: mass 5 -> 3.95; geometry collision box size=0.25 0.25 0.25; visual mesh filename=package://neuronbot2_description/meshes/neuronbot2/base_lin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
- link laser_frame: mass 0.2 -> 0.362
- link wheel_left_link: mass 2.8498940e-02 -> None; geometry collision mesh filename=package://neuronbot2_description/meshes/neuronbot2/wheel_li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; visual mesh filename=package://neuronbot2_description/meshes/neuronbot2/wheel_li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
- link wheel_right_link: mass 2.8498940e-02 -> None; geometry collision mesh filename=package://neuronbot2_description/meshes/neuronbot2/wheel_li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; visual mesh filename=package://neuronbot2_description/meshes/neuronbot2/wheel_li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
Joints:
- joint l_wheel_joint: origin xyz=0.0 0.14 0.0745 rpy=1.57 0 0 -> xyz=0.0 0.109 0.0415 rpy=0 0 0
- joint laser_frame_joint: origin xyz=0.125 0 0.33 rpy=0 0 3.14 -> xyz=0.00254 0 0.227 rpy=0 0 3.14
- joint r_wheel_joint: origin xyz=0.0 -0.14 0.0745 rpy=1.57 0 0 -> xyz=0.0 -0.109 0.0415 rpy=0 0 0

Commit message: Update tf

File: neuronbot2_description/urdf/neuronbot2.urdf (robot description, URDF)
Before this commit: robot neuronbot2_description, 6 links, 5 joints
Links:
- link base_link: mass 3.95 -> 8.3; geometry collision box size=0.25 0.25 0.25; visual mesh filename=package://neuronbot2_description/meshes/neuronbot2/base_lin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 scale=0.001 0.001 0.001
- link laser_frame: geometry collision mesh filename=package://neuronbot2_description/meshes/neuronbot2/laser_li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 scale=0.001 0.001 0.001; visual mesh filename=package://neuronbot2_description/meshes/neuronbot2/laser_li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 scale=0.001 0.001 0.001
- link wheel_left_link: geometry collision mesh filename=package://neuronbot2_description/meshes/neuronbot2/wheel_li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 scale=0.001 0.001 0.001; visual mesh filename=package://neuronbot2_description/meshes/neuronbot2/wheel_li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 scale=0.001 0.001 0.001
- link wheel_right_link: geometry collision mesh filename=package://neuronbot2_description/meshes/neuronbot2/wheel_li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 scale=0.001 0.001 0.001; visual mesh filename=package://neuronbot2_description/meshes/neuronbot2/wheel_li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 scale=0.001 0.001 0.001
Joints:
- joint imu_joint: origin xyz=0 0 0.11 rpy=0 0 0 -> xyz=0.075 0 0.138 rpy=0 0 0
- joint l_wheel_joint: axis 0 0 1 -> 0 1 0
- joint laser_frame_joint: origin xyz=0.00254 0 0.227 rpy=0 0 3.14 -> xyz=0 0 0.205 rpy=0 0 3.14
- joint r_wheel_joint: axis 0 0 1 -> 0 1 0; origin xyz=0.0 -0.109 0.0415 rpy=0 0 0 -> xyz=0.0 -0.109 0.0415 rpy=0 0 3.14

Commit message: Change body color to while for better a demo appearance

File: neuronbot2_description/urdf/neuronbot2.urdf (robot description, URDF)
Before this commit: robot neuronbot2_description, 6 links, 5 joints
Joints:
- joint laser_frame_joint: origin xyz=0 0 0.205 rpy=0 0 3.14 -> xyz=0 0 0.205 rpy=0 0 0

Commit message: Fix urdf model

File: neuronbot2_description/urdf/neuronbot2.urdf (robot description, URDF)
Before this commit: robot neuronbot2_description, 6 links, 5 joints
Joints:
- joint laser_frame_joint: origin xyz=0 0 0.205 rpy=0 0 0 -> xyz=0 0 0.205 rpy=0 0 3.14

Commit message: Update code

File: neuronbot2_description/urdf/neuronbot2.urdf (robot description, URDF)
Before this commit: robot neuronbot2_description, 3 links, 2 joints
Links:
- added link base_footprint
Joints:
- added joint base: type fixed, parent base_footprint, child base_link, origin xyz=0 0 0 rpy=0 0 0

Commit message: Update URDF and stl files for new robots

File: neuronbot2_description/urdf/neuronbot2.urdf (robot description, URDF)
Before this commit: robot neuronbot2_description, 4 links, 3 joints
Links:
- added link wheel_left_link; collision mesh filename=package://neuronbot2_description/meshes/neuronbot2/wheel_li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 scale=0.001 0.001 0.001; visual mesh filename=package://neuronbot2_description/meshes/neuronbot2/wheel_li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 scale=0.001 0.001 0.001
- added link wheel_right_link; collision mesh filename=package://neuronbot2_description/meshes/neuronbot2/wheel_li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 scale=0.001 0.001 0.001; visual mesh filename=package://neuronbot2_description/meshes/neuronbot2/wheel_li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 scale=0.001 0.001 0.001
- link base_link: mass 4.7982 -> 8.3; geometry collision box size=0.25 0.25 0.25; visual mesh filename=package://neuronbot2_description/meshes/neuronbot2/base_lin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 scale=0.001 0.001 0.001
- link laser_frame: mass 0.17934 -> 0.362; geometry collision mesh filename=package://neuronbot2_description/meshes/neuronbot2/laser_li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 scale=0.001 0.001 0.001; visual mesh filename=package://neuronbot2_description/meshes/neuronbot2/laser_li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 scale=0.001 0.001 0.001
Joints:
- removed joint base
- added joint base_link_joint: type fixed, parent base_footprint, child base_link, origin xyz=0 0 0 rpy=0 0 0
- added joint l_wheel_joint: type continuous, parent base_link, child wheel_left_link, origin xyz=0.0 0.109 0.0415 rpy=0 0 0, axis 0 1 0
- added joint r_wheel_joint: type continuous, parent base_link, child wheel_right_link, origin xyz=0.0 -0.109 0.0415 rpy=0 0 3.14, axis 0 1 0
- joint imu_joint: axis (none) -> 0 0 0; origin xyz=0 0 0.11 rpy=0 0 1.57 -> xyz=0.075 0 0.138 rpy=0 0 0
- joint laser_frame_joint: origin xyz=0.001 0 0.31 rpy=0 0 3.14 -> xyz=0 0 0.205 rpy=0 0 3.14

Commit message: Add camera on neruonbot2 simulation.

File: neuronbot2_description/urdf/neuronbot2.urdf (robot description, URDF)
Before this commit: robot neuronbot2_description, 6 links, 5 joints
Links:
- added link camera_link
Joints:
- added joint camera_joint: type fixed, parent base_link, child camera_link, origin xyz=0.075 0 0.250 rpy=0 0 0, axis 0 0 0

Commit message: Tune imu and odom.
1. Base driver pub imu.
2. Add ekf.

File: neuronbot2_description/urdf/neuronbot2.urdf (robot description, URDF)
Before this commit: robot neuronbot2_description, 6 links, 5 joints
Joints:
- joint imu_joint: origin xyz=0.075 0 0.138 rpy=0 0 0 -> xyz=0.075 0 0.138 rpy=0 0 1.57

Commit message: Fix camera orientation

File: neuronbot2_description/urdf/neuronbot2.urdf (robot description, URDF)
Before this commit: robot neuronbot2_description, 7 links, 6 joints
Joints:
- joint camera_joint: origin xyz=0.075 0 0.250 rpy=0 0 0 -> xyz=0.075 0 0.250 rpy=1.570795 3.14159 1.570795

Commit message: Fix Wheels TF display in RVIZ

File: neuronbot2_description/urdf/neuronbot2.urdf (robot description, URDF)
Before this commit: robot neuronbot2_description, 7 links, 6 joints
Joints:
- joint r_wheel_joint: origin xyz=0.0 -0.109 0.0415 rpy=0 0 3.14 -> xyz=0.0 -0.09 0.0415 rpy=0 0 0

Commit message: Change the position of imu_link in URDF and SDF

File: neuronbot2_description/urdf/neuronbot2.urdf (robot description, URDF)
Before this commit: robot neuronbot2_description, 6 links, 5 joints
Joints:
- joint imu_joint: origin xyz=0.075 0 0.138 rpy=0 0 1.57 -> xyz=0 0 -0.05 rpy=0 0 0

Commit message: Add camera config and fine tune STVL

File: neuronbot2_description/urdf/neuronbot2.urdf (robot description, URDF)
Before this commit: robot neuronbot2_description, 6 links, 5 joints
Links:
- added link camera_link; collision box size=0.012 0.132 0.020; visual mesh filename=package://TODO.dae
Joints:
- added joint camera_joint: type fixed, parent base_link, child camera_link, origin xyz=0.175 0.0 0.175 rpy=0 0.1 0

Commit message: Change camera pose elevation

File: neuronbot2_description/urdf/neuronbot2.urdf (robot description, URDF)
Before this commit: robot neuronbot2_description, 7 links, 6 joints
Joints:
- joint camera_joint: origin xyz=0.175 0.0 0.175 rpy=0 0.1 0 -> xyz=0.175 0.0 0.175 rpy=0 0.15 0

Commit message: Fine tune STVL

File: neuronbot2_description/urdf/neuronbot2.urdf (robot description, URDF)
Before this commit: robot neuronbot2_description, 7 links, 6 joints
Joints:
- joint camera_joint: origin xyz=0.175 0.0 0.175 rpy=0 0.15 0 -> xyz=0.175 0.0 0.175 rpy=0 0.10 0

Commit message: Change IMU position

File: neuronbot2_description/urdf/neuronbot2.urdf (robot description, URDF)
Before this commit: robot neuronbot2_description, 7 links, 6 joints
Joints:
- joint imu_joint: origin xyz=0.075 0 0.138 rpy=0 0 0 -> xyz=0.055 -0.010 0.070 rpy=0 0 -1.5708
