Commit message: Fix the simulated camera orientation of '*_optical_frame' according to REP-103

File: neuronbot2_description/urdf/neuronbot2_w_front_camera.urdf (robot description, URDF)
Before this commit: robot neuronbot2_description, 9 links, 8 joints
Links:
- removed link depth_camera_frame
- removed link rgb_camera_frame
- added link camera_color_frame
- added link camera_color_optical_frame
- added link camera_depth_frame
- added link camera_depth_optical_frame
Joints:
- removed joint depth_camera_joint
- removed joint rgb_camera_joint
- added joint camera_color_joint: type fixed, parent camera_link, child camera_color_frame, origin xyz=0 0 0 rpy=0 0 0
- added joint camera_color_optical_joint: type fixed, parent camera_color_frame, child camera_color_optical_frame, origin xyz=0 0 0 rpy=-1.57 0 -1.57
- added joint camera_depth_joint: type fixed, parent camera_link, child camera_depth_frame, origin xyz=0 0 0 rpy=0 0 0
- added joint camera_depth_optical_joint: type fixed, parent camera_depth_frame, child camera_depth_optical_frame, origin xyz=0 0 0 rpy=-1.57 0 -1.57

File: neuronbot2_description/urdf/neuronbot2_w_top_camera.urdf (robot description, URDF)
Before this commit: robot neuronbot2_description, 9 links, 8 joints
Links:
- removed link depth_camera_frame
- removed link rgb_camera_frame
- added link camera_color_frame
- added link camera_color_optical_frame
- added link camera_depth_frame
- added link camera_depth_optical_frame
Joints:
- removed joint depth_camera_joint
- removed joint rgb_camera_joint
- added joint camera_color_joint: type fixed, parent camera_link, child camera_color_frame, origin xyz=0 0 0 rpy=0 0 0
- added joint camera_color_optical_joint: type fixed, parent camera_color_frame, child camera_color_optical_frame, origin xyz=0 0 0 rpy=-1.57 0 -1.57
- added joint camera_depth_joint: type fixed, parent camera_link, child camera_depth_frame, origin xyz=0 0 0 rpy=0 0 0
- added joint camera_depth_optical_joint: type fixed, parent camera_depth_frame, child camera_depth_optical_frame, origin xyz=0 0 0 rpy=-1.57 0 -1.57
